Commit message: Add: Test wrapper node

File: src/arp_resources/arp_deployment_gp20/model/xacro_files/gp20_hl_macro.xacro (robot description, xacro)
@@ -20,5 +20,5 @@
         <visual>
             <geometry>
-                <mesh filename="package://rarp_deployment_gp20/model/mesh_files/visual/link_1_s.stl"/>
+                <mesh filename="package://arp_deployment_gp20/model/mesh_files/visual/link_1_s.stl"/>
             </geometry>
             <xacro:material_yaskawa_blue/>
@@ -95,4 +95,5 @@
         </collision>
     </link>
+    <link name="${prefix}tool0" />
     <!-- end of link list -->
     <!-- joint list -->
@@ -155,5 +156,4 @@
     </joint>
     <!-- ROS-Industrial 'tool0' frame - all-zeros tool frame -->
-    <link name="${prefix}tool0"/>
     <joint name="${prefix}flange-tool0" type="fixed">
       <origin xyz="0 0 0" rpy="${radians(180)} -${radians(90)} 0"/>
